File: Telemetry/Schematics/telem_board.sch (EAGLE design)
At the start: 30 parts, among them IC1 PIC18F26K80I/SP, IC2 PTN78000WAH, IC3 ISO1050DUB, IC4 FT232RL, J1 ICD, J2 TELEM, J3 TELEM, J4 TEMP SENSOR, J5 HALL SENSOR, Q4 20M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

Commit message: telem_boardV2
Parts:
- removed C10: 100n, resistor:C-USC0805
- removed C3, C8: 47p, resistor:C-USC0805
- removed F1: 0.5, MSCP_2011_v2:PTC0ZCA
- removed LED1: (no value), adafruit:LED5MM
- removed X2: +12V, con-phoenix-508:MSTBA2
- added J7: RADIO, con-amp:215877-7
- added TEST: (no value), led:LED5MM
- IC4: value FT232RL -> SN75LBC179D; device MSCP_2011_v2:FT232RL -> MSCP_2011_v1:SN75LBC179D
- J2, J3: value TELEM -> CANBUS
- R2: device rcl:R-US_R0805 -> adafruit:R-US_R0805
- X1: value PN61729-S -> +12V; device con-berg:PN61729-S -> con-phoenix-508:MSTBA2
Connections:
- removed net N$9: C10.1, IC4.3V3OUT
- new net N$12: IC4.Y, J7.1
- net +12V: now also X1-2.1; no longer X2-2.1
- net +5V: now also J7.3, J7.6; no longer F1.1, IC4.!RESET, IC4.VCCIO
- net CTS: no longer IC4.!CTS
- net GND: now also J7.7, J7.8, R2.1, X1-1.1; no longer C10.2, C3.2, C8.2, IC4.GND@1, IC4.GND@2, IC4.GND@A, IC4.TEST, R2.2, X1.4, X2-1.1
- net N$10: now also IC4.Z, J7.2; no longer F1.2, X1.1
- net N$3: now also IC4.B, J7.5; no longer IC1.RB2/CANTX/C1OUT/P1C/CTED1/INT2, LED1.A
- net N$4: now also IC4.A, J7.4; no longer LED1.C, R2.1
- net N$6: now also IC1.RB2/CANTX/C1OUT/P1C/CTED1/INT2, TEST.A; no longer C8.1, IC4.USBDM, X1.2
- net N$7: now also R2.2, TEST.C; no longer C3.1, IC4.USBDP, X1.3
- net RTS: no longer IC4.!RTS
- net RX: now also IC4.R; no longer IC4.TXD
- net TX: now also IC4.D; no longer IC4.RXD
Other:
- moved on the sheet: C11, C12, R2

Commit message: telem_board_v3
Parts:
- removed R10: 100, rcl:R-US_0207/7
- added H2, H3, H4: MOUNT-HOLE2.8, holes:MOUNT-HOLE2.8
- added TERM: 100, resistor:R-EU_0207/10
- J4: value TEMP SENSOR -> HALLSENS
- J5: value HALL SENSOR -> TEMPSENS
Connections:
- removed net N$14: IC3.CANH, J2.5, J3.5, R10.2
- removed net N$15: IC3.CANL, J2.4, J3.4, R10.1
- removed net N$16: IC3.GND2, J2.1, J2.2, J2.3, J3.1, J3.2, J3.3
- removed net N$32: IC3.VCC2, J2.6, J2.7, J2.8, J3.6, J3.7, J3.8
- new net CANH: IC3.CANH, J2.5, J3.5, TERM.1
- new net CANL: IC3.CANL, J2.4, J3.4, TERM.2
- net +12V: now also J2.8, J3.8
- net +5V: now also IC3.VCC2, J2.6, J2.7, J3.6, J3.7
- net GND: now also IC3.GND2, J2.1, J2.2, J2.3, J3.1, J3.2, J3.3
Other:
- moved on the sheet: IC4, J2, J7

Commit message: telem_board_v4
Connections:
- net +12V: now also J2.1, J2.2, J3.1, J3.2; no longer J2.8, J3.8
- net +5V: now also J2.3, J3.3; no longer J2.6, J2.7, J3.6, J3.7
- net CANH: now also J2.4, J3.4; no longer J2.5, J3.5
- net CANL: now also J2.5, J3.5; no longer J2.4, J3.4
- net GND: now also J2.6, J2.7, J2.8, J3.6, J3.7, J3.8; no longer J2.1, J2.2, J2.3, J3.1, J3.2, J3.3

Commit message: telem_board_v6
Parts:
- added R3, R5: (no value), eagle-ltspice:R
Connections:
- removed net CTS: IC1.RB3/CANRX/C1OUT/P1C/CTED1/INT3
- removed net N$18: IC1.RC7/CANRX/RX1/DT1/CCP4, IC3.RXD
- removed net RTS: IC1.RB5/T0CKI/T3CKI/CCP5/KBI1
- new net CAN5V: IC3.VCC2, J2.3, J3.3
- new net CANGND: IC3.GND2, J2.6, J2.7, J2.8, J3.6, J3.7, J3.8
- new net N$9: IC1.RB3/CANRX/C1OUT/P1C/CTED1/INT3, IC3.RXD
- net +5V: now also R3.1, R5.1; no longer IC3.VCC2, J2.3, J3.3
- net GND: no longer IC3.GND2, J2.6, J2.7, J2.8, J3.6, J3.7, J3.8
- net N$11: now also IC1.RB5/T0CKI/T3CKI/CCP5/KBI1, TEST.A; no longer IC1.RC6/CANTX/TX1/CK1/CCP3, IC3.TXD
- net N$6: now also IC3.TXD; no longer TEST.A
- net SCL: now also R3.2
- net SDA: now also R5.2
Other:
- moved on the sheet: C1, C4, C5, H2, H3, H4, IC2, IC3, J2, J3, R1, R2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

Commit message: real telem_board_v6
previous one was v5
Parts:
- removed TERM: 100, resistor:R-EU_0207/10
- removed X1: +12V, con-phoenix-508:MSTBA2
- added DPAK: DIODE_2SCHOTTKY-DPAK, MSCP_2011_v2:DIODE_2SCHOTTKY-DPAK
- added POWER: MSTBA3, con-phoenix-508:MSTBA3
- TEST: device led:LED5MM -> led:LEDCHIP-LED0805
- renumbered J1 to 1
Connections:
- net N$11 renamed STATUS
- removed net CAN5V: IC3.VCC2, J2.3, J3.3
- removed net CANGND: IC3.GND2, J2.6, J2.7, J2.8, J3.6, J3.7, J3.8
- new net N$13: DPAK.A1, POWER-1.1
- new net N$14: DPAK.A2, POWER-2.1
- new net N$15: 1.4, IC1.RB7/PGD/T3G/RX2/DT2/KBI3
- new net N$16: 1.5, IC1.RB6/PGC/PGD/TX2/CK2/KBI2
- net +12V: now also DPAK.C; no longer X1-2.1
- net +5V: now also IC3.VCC2, J2.3, J3.3
- net CANH: no longer TERM.1
- net CANL: no longer TERM.2
- net GND: now also IC3.GND2, J2.6, J2.7, J2.8, J3.6, J3.7, J3.8, POWER-3.1; no longer X1-1.1
- net RX: now also IC1.RC7/CANRX/RX1/DT1/CCP4; no longer 1.4, IC1.RB7/PGD/T3G/RX2/DT2/KBI3
- net TX: now also IC1.RC6/CANTX/TX1/CK1/CCP3; no longer 1.5, IC1.RB6/PGC/PGD/TX2/CK2/KBI2
Other:
- note added: "+12"
- note added: "AUX 12"
- note added: "GND"
- note added: "Start in (Switched AUX battery)"
- moved on the sheet: R2, TEST
